File: module_duplex_sx126x.kicad_sch (KiCad schematic)
At the start: 39 parts, among them J1 USB_B_Mini, J2 Conn_01x06_Pin, J3 Conn_01x05, J4 Conn_01x04, J6 Conn_01x02, SW1 SW_Push, U1 STM32F103C8Tx, U2 AMS1117-3.3, U3 SN65HVD230, U4 Ai-Thinker-Ra-02, U5 Ai-Thinker-Ra-02, Y1 16M, Y2 32.768k

Commit message: Corrected DIO1 BUSY pin in radio module
Signed-off-by: Leonardo Celente <leocelente@gmail.com>
Parts:
- removed U4, U5: Ai-Thinker-Ra-02, RF_Module:Ai-Thinker-Ra-01-LoRa, symbol RF_Module:Ai-Thinker-Ra-02
- added U6, U7: Ai-Thinker-Ra-01SH, RF_Module:Ai-Thinker-Ra-01-LoRa, symbol RF_Module:Ai-Thinker-Ra-01SH
- C13, C14, C9: value 4.7u -> 10u; footprint Capacitor_SMD:C_0603_1608Metric -> Capacitor_SMD:C_0805_2012Metric; LCSC C19666 -> C19702
- C8: value 4.7u -> 0.1u; LCSC C19666 -> C14663
Connections:
- net RADIO_RECV_DIO0 is gone; now on net RADIO_RECV_DIO1: U1.19 (PB1)
- net RADIO_SEND_DIO0 is gone; now on net RADIO_SEND_DIO1: U1.30 (PA9)
- net GND: now also U6.16 (GND), U6.2 (GND), U6.9 (GND), U7.16 (GND), U7.2 (GND), U7.9 (GND)
- net RADIO_RECV_DIO1: now also U7.6 (DIO1); no longer U1.20 (PB2)
- net RADIO_RECV_MISO: now also U7.13 (MISO)
- net RADIO_RECV_MOSI: now also U7.14 (MOSI)
- net RADIO_RECV_NSS: now also U7.15 (~{NSS})
- net RADIO_RECV_RST: now also U7.4 (~{RESET})
- net RADIO_RECV_SCK: now also U7.12 (SCK)
- net RADIO_SEND_DIO1: now also U6.6 (DIO1); no longer U1.31 (PA10)
- net RADIO_SEND_MISO: now also U6.13 (MISO)
- net RADIO_SEND_MOSI: now also U6.14 (MOSI)
- net RADIO_SEND_NSS: now also U6.15 (~{NSS})
- net RADIO_SEND_RST: now also U6.4 (~{RESET})
- net RADIO_SEND_SCK: now also U6.12 (SCK)
- net VCC: now also U6.3 (VDD), U7.3 (VDD)
- new net RADIO_RECV_BUSY: U1.20 (PB2), U7.10 (BUSY)
- new net RADIO_SEND_BUSY: U1.31 (PA10), U6.10 (BUSY)
- no-connect marks 12 -> 14

Commit message: Updated Production and added README
Signed-off-by: Leonardo Celente <leocelente@gmail.com>
Parts:
- U6, U7: now left out of the parts list
Changed lines of the file:
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@@
   )
   (symbol (lib_id "RF_Module:Ai-Thinker-Ra-01SH") (at 229.87 138.43 0) (unit 1)
-    (in_bom yes) (on_board yes) (dnp no) (fields_autoplaced)
+    (in_bom no) (on_board yes) (dnp no) (fields_autoplaced)
     (property "Reference" "U6" (at 231.8259 121.92 0)
       (effects (font (size 1.27 1.27)) (justify left))
@@
     )
     (property "Datasheet" "http://wiki.ai-thinker.com/_media/lora/docs/c047ps01a1_ra-01_product_specification_v1.1.pdf" (at 232.41 120.65 0)
+      (effects (font (size 1.27 1.27)) hide)
+    )
+    (property "Aoba" "" (at 229.87 138.43 0)
       (effects (font (size 1.27 1.27)) hide)
     )
@@
   )
   (symbol (lib_id "RF_Module:Ai-Thinker-Ra-01SH") (at 229.87 81.28 0) (unit 1)
-    (in_bom yes) (on_board yes) (dnp no) (fields_autoplaced)
+    (in_bom no) (on_board yes) (dnp no) (fields_autoplaced)
     (property "Reference" "U7" (at 231.8259 64.77 0)
       (effects (font (size 1.27 1.27)) (justify left))
@@
       (effects (font (size 1.27 1.27)) hide)
     )
+    (property "Aoba" "" (at 229.87 81.28 0)
+      (effects (font (size 1.27 1.27)) hide)
+    )
